File: Eurorack VCA/Eurorack VCA motherboard.sch (KiCad schematic (older format))
At the start: 22 parts, among them J1 JACK_MONO_SW, J2 JACK_MONO_SW, J3 JACK_MONO_SW, J4 JACK_MONO_SW, J5 JACK_MONO_SW, J6 JACK_MONO_SW, P1 50K, P2 50K, P3 50K, P4 50K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

Commit message: fixed Eurorack VCA CV gain pot. Was reversed. Now v1.1. Ordered updated PCBs from DirtyPCBs.com
Connections:
- net CV1A: now also P3.3; no longer P3.1
- net CV2A: now also P6.3; no longer P6.1
- net at R2.2, U1.2 (-): now also P3.1; no longer P3.3
- net at R4.2, U1.6 (-): now also P6.1; no longer P6.3
Changed lines of the file:
@@
 LIBS:MySynthParts
 LIBS:Eurorack VCA motherboard-cache
-EELAYER 27 0
+EELAYER 24 0
 EELAYER END
 $Descr A4 11693 8268
@@
 F 3 "~" H 9650 5800 60  0000 C CNN
 	1    9650 5800
-	-1   0    0    -1
+	1    0    0    -1
 $EndComp
 Wire Wire Line
@@
 F 3 "~" H 4150 5400 60  0000 C CNN
 	1    4150 5400
-	-1   0    0    -1
-$EndComp
-Wire Wire Line
+	1    0    0    -1
+$EndComp
+Wire Wire Line
